File: eagle/adon3AA.brd (EAGLE design)
At the start: 56.8 x 47 mm, 22 parts

Commit message: board design is done
Parts:
- removed C1: 10uF, SparkFun-Capacitors:CPOL-RADIAL-10UF-25V
- added C3: 10uF, SparkFun-Capacitors:CPOL-RADIAL-10UF-25V
- added ICSP: (no value), SparkFun-Connectors:2X3-NS
- added R1: 10k, SparkFun-Resistors:AXIAL-0.4
- added S2: SOUND, SparkFun-Electromechanical:SWITCH-SPDT_LOCK.007S
- LED1: value Green -> BLUE
- LED2: value Red -> YELLOW
- LED3: value Yellow -> RED
- LED4: value Blue -> GREEN
- R16: value 150 -> 220
- SW1: device special:EDG-03 -> special:EDG-02
- moved LED4 92.2 mm to (50.8, 20.3)
- moved LED3 82.7 mm to (35.6, 20.3)
- moved ATTINY84 78.0 mm to (48.3, 35.6), turned to 270 degrees
- moved BUZZER 70.4 mm to (24.1, 35.6)
- moved PWRLED 69.5 mm to (20.3, 43.2), turned to 180 degrees
- moved LED1 66.0 mm to (5.08, 20.3)
- moved C2 56.4 mm to (38.1, 34.3), turned to 90 degrees
- moved SW1 56.1 mm to (14.0, 40.6)
- moved LED2 55.0 mm to (20.3, 20.3)
- moved BATTERY 29.3 mm to (31.8, 40.6), turned to 0 degrees
- moved S1 21.6 mm to (2.54, 40.6)
- moved R16 17.8 mm to (29.2, 12.7), turned to 270 degrees
- moved R15 15.3 mm to (44.5, 12.7), turned to 270 degrees
- moved R8 15.3 mm to (11.4, 12.7)
- moved R6 15.3 mm to (26.7, 12.7), turned to 270 degrees
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Connections:
- new net N$21: ATTINY84.4, ICSP.5, R1.P$1
- net GND: now also C3.2, ICSP.6, S2.3, SW1.3; no longer C1.2, SW1.5, SW1.6
- net N$10: now also SW1.1; no longer SW1.2
- net N$11: now also SW1.2; no longer SW1.3
- net N$13: now also ICSP.1
- net N$14: now also ICSP.3
- net N$23: now also S2.2; no longer SW1.1
- net N$9: now also ICSP.4
- net VCC: now also C3.1, ICSP.2, R1.P$2; no longer ATTINY84.4, C1.1
Routing:
- net N$14: track 0.00 -> 102.9 mm
- net VCC: track 0.00 -> 99.3 mm
- net N$13: track 0.00 -> 85.0 mm, vias 0 -> 1
- net N$15: track 0.00 -> 70.9 mm
- net N$9: track 0.00 -> 69.8 mm
- net N$21: track 0.00 -> 67.9 mm, vias 0 -> 1
- net N$16: track 0.00 -> 60.9 mm, vias 0 -> 2
- net N$5: track 0.00 -> 52.1 mm, vias 0 -> 1
- net N$10: track 0.00 -> 44.8 mm, vias 0 -> 1
- net N$6: track 0.00 -> 41.0 mm
- net N$18: track 0.00 -> 33.9 mm
- net N$11: track 0.00 -> 32.1 mm, vias 0 -> 1
- net N$12: track 0.00 -> 30.3 mm
- net N$2: track 0.00 -> 29.0 mm
- net N$17: track 0.00 -> 28.8 mm
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- added copper zone on layer 1, net GND
- added copper zone on layer 16, net GND
Other:
- board text added: "Adon v4 arolsen@gmail.com"
