File: eagle/adon3AA.sch (EAGLE design)
At the start: 22 parts

Commit message: board design is done
Parts:
- removed C1: 10uF, SparkFun-Capacitors:CAP_POLPTH2
- added C3: 10uF, SparkFun-Capacitors:CAP_POLPTH2
- added ICSP: (no value), SparkFun-Connectors:M03X2NO_SILK
- added R1: 10k, SparkFun-Resistors:RESISTORPTH-1/4W
- added S2: SOUND, SparkFun-Electromechanical:SWITCH-SPDTPTH_LOCK
- LED1: value Green -> BLUE
- LED2: value Red -> YELLOW
- LED3: value Yellow -> RED
- LED4: value Blue -> GREEN
- R16: value 150 -> 220
- SW1: device special:SW_DIP-3 -> special:SW_DIP-2
Connections:
- new net N$21: ATTINY84.(PCINT11/~RESET/DW)PB3, ICSP.5, R1.1
- net GND: now also C3.-, ICSP.6, S2.S, SW1.3; no longer C1.-, SW1.5, SW1.6
- net N$10: now also SW1.1; no longer SW1.2
- net N$11: now also SW1.2; no longer SW1.3
- net N$13: now also ICSP.1
- net N$14: now also ICSP.3
- net N$23: now also S2.P; no longer SW1.1
- net N$9: now also ICSP.4
- net VCC: now also C3.+, ICSP.2, R1.2; no longer ATTINY84.(PCINT11/~RESET/DW)PB3, C1.+
